Commit message: fix: align robot dimensions with spec and add gazebo plugin interface

File: src/diy_nav_description/urdf/diy_nav_bot.urdf.xacro (robot description, xacro)
@@ -20,3 +20,5 @@
   <xacro:include filename="$(find diy_nav_description)/urdf/wheels.xacro"/>
   <xacro:include filename="$(find diy_nav_description)/urdf/sensors.xacro"/>
+  <!-- Gazebo 插件与物理属性（阶段 4.5 为空壳，阶段 5 填充实现） -->
+  <xacro:include filename="$(find diy_nav_description)/urdf/gazebo_plugins.xacro"/>
 </robot>

File: src/diy_nav_description/urdf/properties.xacro (robot description, xacro)
@@ -7,5 +7,5 @@
   尺寸设计目标：
     - 室内两轮差速移动机器人
-    - 低矮矩形底盘 + 上盖 + 左右驱动轮 + 后方球形万向轮
+    - 低矮矩形底盘 + 上盖 + 左右驱动轮 + 前方球形万向轮
     - 顶部二维激光雷达（安装于圆柱底座）+ 底盘中心 IMU 盒体
   坐标约定（ROS REP-103）：
@@ -21,7 +21,7 @@
        底盘主体（chassis）
        ============================================================ -->
-  <!-- 主底盘长（x）×宽（y）×高（z） -->
-  <xacro:property name="base_length" value="0.46"/>
-  <xacro:property name="base_width"  value="0.34"/>
+  <!-- 主底盘长（x）×宽（y）×高（z）；0.45×0.32 对齐规格书 -->
+  <xacro:property name="base_length" value="0.45"/>
+  <xacro:property name="base_width"  value="0.32"/>
   <xacro:property name="base_height" value="0.12"/>
   <xacro:property name="base_mass"   value="8.0"/>
@@ -35,5 +35,6 @@
   <xacro:property name="upper_length" value="0.38"/>
   <xacro:property name="upper_width"  value="0.28"/>
-  <xacro:property name="upper_height" value="0.08"/>
+  <!-- 上盖高度 0.02：从 0.08 收薄，配合激光底座使扫描平面精确落到 0.23 m -->
+  <xacro:property name="upper_height" value="0.02"/>
   <xacro:property name="upper_mass"   value="1.5"/>
   <!-- ============================================================
@@ -43,15 +44,16 @@
   <xacro:property name="wheel_width"      value="0.035"/>
   <xacro:property name="wheel_mass"       value="0.60"/>
-  <!-- 左右轮中心距（沿 y 轴） -->
-  <xacro:property name="wheel_separation" value="0.31"/>
+  <!-- 左右轮中心距（沿 y 轴）= 0.36：轮外缘 y=0.1975 > 底盘半宽 0.16，
+       轮子完整探出底盘侧面，消除埋入底盘的物理隐患 -->
+  <xacro:property name="wheel_separation" value="0.36"/>
   <!-- 轮心沿 x 方向偏移（0 表示位于底盘几何中心正下方） -->
   <xacro:property name="wheel_x_offset"   value="0.0"/>
   <!-- ============================================================
-       后万向轮（球体近似）
+       前万向轮（球体近似）
        ============================================================ -->
   <xacro:property name="caster_radius" value="0.035"/>
   <xacro:property name="caster_mass"   value="0.15"/>
-  <!-- caster 相对底盘中心的 x 位置（负值表示后方） -->
-  <xacro:property name="caster_x_offset" value="-0.16"/>
+  <!-- caster 相对底盘中心的 x 位置（正值表示前方，规格书要求 front_caster） -->
+  <xacro:property name="caster_x_offset" value="0.16"/>
   <!-- ============================================================
        激光雷达（顶部）
@@ -59,7 +61,11 @@
   <!-- 圆柱底座尺寸 -->
   <xacro:property name="laser_mount_radius" value="0.045"/>
-  <xacro:property name="laser_mount_height" value="0.035"/>
+  <!-- 底座高度 0.01：与收薄的上盖配合，使 laser_link 原点离地精确 = 0.23 m -->
+  <xacro:property name="laser_mount_height" value="0.01"/>
   <xacro:property name="laser_mount_mass"   value="0.20"/>
-  <!-- 激光扫描平面（laser_link 原点）相对地面高度目标 ~0.265 m
+  <!-- 激光扫描平面（laser_link 原点）相对地面高度目标 = 0.23 m（规格：约 0.23）
+       0.23 = base_link_z_offset (0.135)
+            + base_height/2 (0.06) + upper_height (0.02)
+            + laser_mount_height (0.01) + laser_link_height/2 (0.005)
        laser_link 位于 laser_mount 顶面上方 -->
   <xacro:property name="laser_link_radius" value="0.030"/>

File: src/diy_nav_description/urdf/wheels.xacro (robot description, xacro)
@@ -3,5 +3,5 @@
   diy_nav_bot / wheels.xacro
   ===========================
-  左右驱动轮（continuous）和后万向轮（球体近似，fixed）。
+  左右驱动轮（continuous）和前万向轮（球体近似，fixed）。
   轮子几何设计：
     - <cylinder> 的默认轴向沿 z；为了让轮子转轴沿 y（机器人左右方向），
@@ -17,5 +17,5 @@
     但由于我们让 base_link 位于底盘中心而非底盘底面，最直接的做法是
     让轮子中心沿 z 方向偏移 -(base_height/2) —— 见 origin 设置。
-  尺寸：wheel_radius=0.075, wheel_width=0.035, wheel_separation=0.31
+  尺寸：wheel_radius=0.075, wheel_width=0.035, wheel_separation=0.36
 -->
 <robot xmlns:xacro="http://www.ros.org/wiki/xacro">
@@ -58,8 +58,9 @@
   <xacro:diy_wheel prefix="left"  y_sign="1"/>
   <xacro:diy_wheel prefix="right" y_sign="-1"/>
-  <!-- ========== 后万向轮（球体近似，fixed joint） ==========
-       本阶段仅作为静态外观和坐标参考；后续 Gazebo 物理仿真阶段
-       会根据摩擦和接触测试重新评估是否需要真实自由度。 -->
-  <link name="rear_caster_link">
+  <!-- ========== 前万向轮（球体近似，fixed joint） ==========
+       位于底盘前部（caster_x_offset=+0.16，规格书要求 front_caster）。
+       球体与地面接触点 z=0，与轮子底面严格共面、无悬空；
+       Gazebo 物理仿真阶段配置零摩擦使其能随车体原地旋转。 -->
+  <link name="front_caster_link">
     <visual>
       <origin xyz="0 0 0" rpy="0 0 0"/>
@@ -82,8 +83,8 @@
   </link>
   <!-- caster 球心 z 相对 base_link = -(base_link_z_offset - caster_radius)
-       即让球心离地 = caster_radius。 -->
-  <joint name="rear_caster_joint" type="fixed">
+       即让球心离地 = caster_radius（球底精确贴地，零悬空）。 -->
+  <joint name="front_caster_joint" type="fixed">
     <parent link="base_link"/>
-    <child  link="rear_caster_link"/>
+    <child  link="front_caster_link"/>
     <origin
       xyz="${caster_x_offset} 0 ${-(base_link_z_offset - caster_radius)}"
