Commit message: feat: integrate DIY robot with Gazebo Classic 11 simulation

File: src/diy_nav_description/urdf/gazebo_plugins.xacro (robot description, xacro)
@@ -3,32 +3,171 @@
   diy_nav_bot / gazebo_plugins.xacro
   ==================================
-  阶段 4.5：本文件为「空壳 + 接口约定」，仅声明阶段 5 将接入的 Gazebo 插件接口。
-  具体 <gazebo> 标签、插件 XML、摩擦与材质映射在阶段 5 填充（届时本文件随
-  validate_description.sh 的阶段参数解锁校验，stage 参数 >= 5 时放行）。
-  阶段 5 接口约定（与 config/gazebo_params.yaml、simulation.launch.py、
-  validate_simulation.sh 保持一致；改动前先同步更新本注释与相关文档）：
-  1. 差速驱动插件（左右轮 continuous joint）
-     - 左轮关节 left_wheel_joint / 右轮关节 right_wheel_joint
-     - wheel_separation = 0.36 m，wheel_diameter = 0.15 m
-     - odometry_frame = odom，robot_base_frame = base_footprint
-     - publish_odom = true，publish_odom_tf = true，publish_wheel_tf = false
-       （odom → base_footprint 全项目唯一 TF 来源；车轮 TF 由 robot_state_publisher 发布）
-     - 更新率 30 Hz；含轮距/轮径/速度与加速度上限等可调参数（集中在 YAML）
-  2. 关节状态发布插件
-     - 输出 /joint_states，覆盖左右驱动轮（供 RSP 发布 wheel TF）
-  3. 2D 激光雷达（<sensor type="ray"> + 对应 ray 传感器插件）
-     - 720 samples，角度范围 -pi ~ +pi，10 Hz
-     - 量程 0.12 ~ 8.0 m，高斯噪声 sigma = 0.01
-     - frame_name = laser_link，输出 sensor_msgs/LaserScan → /scan
-  4. IMU（<sensor type="imu"> + 对应 IMU 传感器插件）
-     - 50 Hz，frame_name = imu_link → /imu
-  5. 接触摩擦（<gazebo reference>）
-     - 左右轮：mu1 = mu2 = 1.0，kp = 1e6，kd = 100
-     - 前万向轮 front_caster_link：mu1 = mu2 = 0.0（fixed caster 零摩擦才能原地旋转）
-  6. 材质映射
-     - materials.xacro 的 6 种 RGBA 颜色 → <gazebo reference> 材质（含透明度）
-  7. 全部节点统一 use_sim_time = true；TF 单一来源，不发布静态 map/odom 冒充。
+  阶段 5：Gazebo Classic 11 插件与物理属性实现。
+  阶段 4.5 曾以空壳形式声明接口，本节内容与之逐项对应：
+    1. 差速驱动插件（模型级）→ /cmd_vel /odom + odom → base_footprint TF
+    2. 关节状态发布插件     → /joint_states（左右驱动轮）
+    3. 2D 激光雷达          → /scan（720 samples / 10 Hz / 0.12~8.0 m / σ=0.01）
+    4. IMU                  → /imu（50 Hz）
+    5. 接触摩擦：轮 mu=1.0，前万向轮 mu=0（fixed caster 零摩擦才能原地旋转）
+    6. 材质映射：6 种 RGBA 颜色 → Gazebo 内置材质
+  约定：
+    - odom → base_footprint 全项目唯一 TF 来源（publish_wheel_tf=false，
+      车轮 TF 由 robot_state_publisher 从 /joint_states 发布，不重复）
+    - 全部数值可调参数集中在本文件顶部属性 + config/gazebo_params.yaml（两处同步）
 -->
 <robot xmlns:xacro="http://www.ros.org/wiki/xacro">
-  <!-- 阶段 5 在此填充 Gazebo 插件与物理属性 -->
+  <!-- ============================================================
+       可调参数（修改时同步 config/gazebo_params.yaml）
+       ============================================================ -->
+  <xacro:property name="diff_drive_update_rate"   value="30"/>
+  <xacro:property name="max_wheel_torque"         value="20"/>
+  <xacro:property name="max_wheel_acceleration"   value="5.0"/>
+  <xacro:property name="joint_state_update_rate"  value="30"/>
+  <xacro:property name="laser_update_rate"        value="10"/>
+  <xacro:property name="laser_samples"            value="720"/>
+  <xacro:property name="laser_min_range"          value="0.12"/>
+  <xacro:property name="laser_max_range"          value="8.0"/>
+  <xacro:property name="laser_noise_stddev"       value="0.01"/>
+  <xacro:property name="imu_update_rate"          value="50"/>
+  <!-- ============================================================
+       1. 差速驱动插件
+       ============================================================ -->
+  <gazebo>
+    <plugin name="diy_diff_drive" filename="libgazebo_ros_diff_drive.so">
+      <ros>
+        <remapping>cmd_vel:=cmd_vel</remapping>
+      </ros>
+      <left_joint>left_wheel_joint</left_joint>
+      <right_joint>right_wheel_joint</right_joint>
+      <wheel_separation>${wheel_separation}</wheel_separation>
+      <wheel_diameter>${2 * wheel_radius}</wheel_diameter>
+      <max_wheel_torque>${max_wheel_torque}</max_wheel_torque>
+      <max_wheel_acceleration>${max_wheel_acceleration}</max_wheel_acceleration>
+      <odometry_frame>odom</odometry_frame>
+      <robot_base_frame>base_footprint</robot_base_frame>
+      <publish_odom>true</publish_odom>
+      <publish_odom_tf>true</publish_odom_tf>
+      <publish_wheel_tf>false</publish_wheel_tf>
+      <update_rate>${diff_drive_update_rate}</update_rate>
+    </plugin>
+  </gazebo>
+  <!-- ============================================================
+       2. 关节状态发布插件（仅左右驱动轮，避免固定关节刷屏）
+       ============================================================ -->
+  <gazebo>
+    <plugin name="diy_joint_state" filename="libgazebo_ros_joint_state_publisher.so">
+      <ros>
+        <remapping>~/out:=joint_states</remapping>
+      </ros>
+      <update_rate>${joint_state_update_rate}</update_rate>
+      <joint_name>left_wheel_joint</joint_name>
+      <joint_name>right_wheel_joint</joint_name>
+    </plugin>
+  </gazebo>
+  <!-- ============================================================
+       3. 2D 激光雷达（安装在 laser_link，360° 全向扫描）
+       ============================================================ -->
+  <gazebo reference="laser_link">
+    <sensor type="ray" name="diy_laser">
+      <pose>0 0 0 0 0 0</pose>
+      <update_rate>${laser_update_rate}</update_rate>
+      <visualize>false</visualize>
+      <ray>
+        <scan>
+          <horizontal>
+            <samples>${laser_samples}</samples>
+            <resolution>1</resolution>
+            <min_angle>-3.141592653589793</min_angle>
+            <max_angle>3.141592653589793</max_angle>
+          </horizontal>
+        </scan>
+        <range>
+          <min>${laser_min_range}</min>
+          <max>${laser_max_range}</max>
+          <resolution>0.01</resolution>
+        </range>
+        <noise>
+          <type>gaussian</type>
+          <mean>0.0</mean>
+          <stddev>${laser_noise_stddev}</stddev>
+        </noise>
+      </ray>
+      <plugin name="diy_laser_plugin" filename="libgazebo_ros_ray_sensor.so">
+        <ros>
+          <remapping>~/out:=scan</remapping>
+        </ros>
+        <output_type>sensor_msgs/LaserScan</output_type>
+        <frame_name>laser_link</frame_name>
+      </plugin>
+    </sensor>
+  </gazebo>
+  <!-- ============================================================
+       4. IMU（安装在 imu_link，底盘几何中心）
+       ============================================================ -->
+  <gazebo reference="imu_link">
+    <sensor type="imu" name="diy_imu">
+      <pose>0 0 0 0 0 0</pose>
+      <!-- always_on 必须显式置 true（官方示例注明 required），否则不触发更新 -->
+      <always_on>true</always_on>
+      <update_rate>${imu_update_rate}</update_rate>
+      <plugin name="diy_imu_plugin" filename="libgazebo_ros_imu_sensor.so">
+        <ros>
+          <remapping>~/out:=imu</remapping>
+        </ros>
+        <update_rate>${imu_update_rate}</update_rate>
+        <frame_name>imu_link</frame_name>
+        <initial_orientation_as_reference>false</initial_orientation_as_reference>
+      </plugin>
+    </sensor>
+  </gazebo>
+  <!-- ============================================================
+       5. 接触摩擦
+       轮子：高摩擦保证驱动；前万向轮：零摩擦（fixed caster 只有零摩擦
+       才能随车体原地旋转，否则车体会被其"别住"）
+       ============================================================ -->
+  <gazebo reference="left_wheel_link">
+    <mu1>1.0</mu1>
+    <mu2>1.0</mu2>
+    <kp>1000000.0</kp>
+    <kd>100.0</kd>
+  </gazebo>
+  <gazebo reference="right_wheel_link">
+    <mu1>1.0</mu1>
+    <mu2>1.0</mu2>
+    <kp>1000000.0</kp>
+    <kd>100.0</kd>
+  </gazebo>
+  <gazebo reference="front_caster_link">
+    <mu1>0.0</mu1>
+    <mu2>0.0</mu2>
+    <kp>1000000.0</kp>
+    <kd>100.0</kd>
+  </gazebo>
+  <!-- ============================================================
+       6. 材质映射（materials.xacro 的 6 种 RGBA → Gazebo 内置材质）
+       ============================================================ -->
+  <gazebo reference="chassis_link">
+    <material>Gazebo/Blue</material>
+  </gazebo>
+  <gazebo reference="upper_body_link">
+    <material>Gazebo/DarkGrey</material>
+  </gazebo>
+  <gazebo reference="left_wheel_link">
+    <material>Gazebo/Black</material>
+  </gazebo>
+  <gazebo reference="right_wheel_link">
+    <material>Gazebo/Black</material>
+  </gazebo>
+  <gazebo reference="front_caster_link">
+    <material>Gazebo/Black</material>
+  </gazebo>
+  <gazebo reference="laser_mount_link">
+    <material>Gazebo/Grey</material>
+  </gazebo>
+  <gazebo reference="laser_link">
+    <material>Gazebo/Orange</material>
+  </gazebo>
+  <gazebo reference="imu_link">
+    <material>Gazebo/Red</material>
+  </gazebo>
 </robot>

File: src/diy_nav_description/urdf/properties.xacro (robot description, xacro)
@@ -47,6 +47,9 @@
        轮子完整探出底盘侧面，消除埋入底盘的物理隐患 -->
   <xacro:property name="wheel_separation" value="0.36"/>
-  <!-- 轮心沿 x 方向偏移（0 表示位于底盘几何中心正下方） -->
-  <xacro:property name="wheel_x_offset"   value="0.0"/>
+  <!-- 轮轴沿 x 的偏移 = -0.04（轮线在质心后方 4.2 cm）：
+       质心几乎落在底盘几何中心，若轮线在质心正下方，前 caster 仅承重 ~1%，
+       机器人处于临界稳定——任何扰动都会后翻到底盘后缘着地（实测 19.5° 倾倒）。
+       轮线后移后 caster 承重 ~18%，俯仰稳定容差 ~15°，水平状态才真正稳定。 -->
+  <xacro:property name="wheel_x_offset"   value="-0.04"/>
   <!-- ============================================================
        前万向轮（球体近似）
@@ -54,6 +57,8 @@
   <xacro:property name="caster_radius" value="0.035"/>
   <xacro:property name="caster_mass"   value="0.15"/>
-  <!-- caster 相对底盘中心的 x 位置（正值表示前方，规格书要求 front_caster） -->
-  <xacro:property name="caster_x_offset" value="0.16"/>
+  <!-- caster 相对底盘中心的 x 位置（正值表示前方，规格书要求 front_caster）
+       0.19 = 底盘半长 0.225 - caster 半径 0.035：球体前缘与底盘前缘齐平，
+       尽量前移以加大与轮线的距离，分担更多车重 -->
+  <xacro:property name="caster_x_offset" value="0.19"/>
   <!-- ============================================================
        激光雷达（顶部）

Commit message: fix: harden wheel contacts and filter laser self-occlusion for map quality

File: src/diy_nav_description/urdf/gazebo_plugins.xacro (robot description, xacro)
@@ -98,5 +98,6 @@
       <plugin name="diy_laser_plugin" filename="libgazebo_ros_ray_sensor.so">
         <ros>
-          <remapping>~/out:=scan</remapping>
+          <!-- 输出到 /scan_raw：scan_filter 过滤车体自遮挡后重发 /scan -->
+          <remapping>~/out:=scan_raw</remapping>
         </ros>
         <output_type>sensor_msgs/LaserScan</output_type>
@@ -127,23 +128,26 @@
        5. 接触摩擦
        轮子：高摩擦保证驱动；前万向轮：零摩擦（fixed caster 只有零摩擦
-       才能随车体原地旋转，否则车体会被其"别住"）
+       才能随车体原地旋转，否则车体会被其"别住"）。
+       kp=1e8/kd=1 为 ODE 默认接触刚度：软接触（1e6）会让车体在碰撞/
+       急转时晃动甚至倾覆（阶段 9 排障记录：急转擦墙后机器人侧翻，
+       车体灌入激光平面污染地图）。
        ============================================================ -->
   <gazebo reference="left_wheel_link">
     <mu1>1.0</mu1>
     <mu2>1.0</mu2>
-    <kp>1000000.0</kp>
-    <kd>100.0</kd>
+    <kp>100000000.0</kp>
+    <kd>1.0</kd>
   </gazebo>
   <gazebo reference="right_wheel_link">
     <mu1>1.0</mu1>
     <mu2>1.0</mu2>
-    <kp>1000000.0</kp>
-    <kd>100.0</kd>
+    <kp>100000000.0</kp>
+    <kd>1.0</kd>
   </gazebo>
   <gazebo reference="front_caster_link">
     <mu1>0.0</mu1>
     <mu2>0.0</mu2>
-    <kp>1000000.0</kp>
-    <kd>100.0</kd>
+    <kp>100000000.0</kp>
+    <kd>1.0</kd>
   </gazebo>
   <!-- ============================================================

File: src/diy_nav_description/urdf/properties.xacro (robot description, xacro)
@@ -33,7 +33,10 @@
        底盘上盖（upper body）
        ============================================================ -->
-  <xacro:property name="upper_length" value="0.38"/>
-  <xacro:property name="upper_width"  value="0.28"/>
-  <!-- 上盖高度 0.02：从 0.08 收薄，配合激光底座使扫描平面精确落到 0.23 m -->
+  <xacro:property name="upper_length" value="0.24"/>
+  <xacro:property name="upper_width"  value="0.20"/>
+  <!-- 上盖高度 0.02：从 0.08 收薄，配合激光底座使扫描平面精确落到 0.23 m
+       长宽 0.24×0.20：边缘距中心 0.10~0.12 m，落入激光盲区（过滤阈值 0.16 m）
+       内——运动俯仰时上盖边缘不再进入扫描平面（阶段 9 排障记录：
+       原 0.38×0.28 上盖边缘 0.14~0.19 m 持续产生自遮挡读数污染地图） -->
   <xacro:property name="upper_height" value="0.02"/>
   <xacro:property name="upper_mass"   value="1.5"/>
