Commit message: fix: save open-doorway map via deterministic saver; stabilize wheel line at -0.08
- map_saver_cli 偶发 'Failed to spin map subscription' 且落盘滞后 → 新增
  scripts/save_map.py（transient_local 直取 /map latch，格式与 map_saver 兼容）
- 重新保存 complex_world 地图：四门口占用 R1 8%/R2 6%/R3 7%/R4 10%
  （旧图 29-43%），走廊中心带 1%，导航可用
- 更新预览图与 yaml
- properties.xacro: 轮线 -0.04 → -0.08（前翻角 15.7° → 28.7°）

File: src/diy_nav_description/urdf/properties.xacro (robot description, xacro)
@@ -50,9 +50,11 @@
        轮子完整探出底盘侧面，消除埋入底盘的物理隐患 -->
   <xacro:property name="wheel_separation" value="0.36"/>
-  <!-- 轮轴沿 x 的偏移 = -0.04（轮线在质心后方 4.2 cm）：
-       质心几乎落在底盘几何中心，若轮线在质心正下方，前 caster 仅承重 ~1%，
-       机器人处于临界稳定——任何扰动都会后翻到底盘后缘着地（实测 19.5° 倾倒）。
-       轮线后移后 caster 承重 ~18%，俯仰稳定容差 ~15°，水平状态才真正稳定。 -->
-  <xacro:property name="wheel_x_offset"   value="-0.04"/>
+  <!-- 轮轴沿 x 的偏移 = -0.08（轮线在质心后方 8.2 cm）：
+       稳定裕度设计（阶段 9 排障记录）：
+       - 0.04 版：质心距轮线 4.2 cm，前翻角 atan(0.042/0.15)≈15.7°——
+         实测减速/冲击即前翻（车体入激光平面污染地图、导航时倾覆）
+       - 0.08 版：质心距轮线 8.2 cm，前翻角 ≈28.7°，caster 承重 ~30%，
+         动态稳定性显著提升；外观上轮子略微后移，仍在底盘下方 -->
+  <xacro:property name="wheel_x_offset"   value="-0.08"/>
   <!-- ============================================================
        前万向轮（球体近似）
